Commit message: minor changes in ddbot_gazebo, and new package ddbot_teleop, that allows user to control robot with virtual joystick

File: ros2_ws/src/ddbot_gazebo/urdf/ddbot.gazebo.xacro (robot description, xacro)
@@ -2,170 +2,11 @@
 <robot xmlns:xacro="http://www.ros.org/wiki/xacro">
     <gazebo>
-        <plugin filename="ignition-gazebo-sensors-system" name="ignition::gazebo::systems::Sensors">
-            <render_engine>ogre2</render_engine>
-        </plugin>
-        <plugin filename="ignition-gazebo-imu-system" name="ignition::gazebo::systems::Imu">
-        </plugin>
         <plugin filename="ignition-gazebo-joint-state-publisher-system"
             name="ignition::gazebo::systems::JointStatePublisher">
         </plugin>
     </gazebo>
-    <!-- Skid Drive -->
-    <gazebo>
-        <plugin filename="ignition-gazebo-diff-drive-system"
-            name="ignition::gazebo::systems::DiffDrive">
-            <left_joint>wheel_fl_joint</left_joint>
-            <right_joint>wheel_fr_joint</right_joint>
-            <left_joint>wheel_rl_joint</left_joint>
-            <right_joint>wheel_rr_joint</right_joint>
-            <wheel_separation>${base_w+wheel_l}</wheel_separation>
-            <wheel_radius>${wheel_r}</wheel_radius>
-            <odom_publish_frequency>30</odom_publish_frequency>
-            <topic>/cmd_vel</topic>
-            <xacro:if value="${odometry_source == 'encoders'}">
-                <odom_topic>$(arg wheel_odom_topic)</odom_topic>
-                <tf_topic>/tf</tf_topic>
-            </xacro:if>
-            <max_wheel_torque>5</max_wheel_torque>
-            <max_wheel_acceleration>0.5</max_wheel_acceleration>
-            <frame_id>odom</frame_id>
-            <child_frame_id>base_footprint</child_frame_id>
-        </plugin>
-    </gazebo>
-    <!-- Ground Truth Odometry -->
-    <xacro:if value="${odometry_source == 'world'}">
-        <gazebo>
-            <plugin filename="libignition-gazebo6-odometry-publisher-system"
-                name="ignition::gazebo::systems::OdometryPublisher">
-                <odom_frame>odom</odom_frame>
-                <robot_base_frame>base_footprint</robot_base_frame>
-                <odom_topic>$(arg wheel_odom_topic)</odom_topic>
-                <tf_topic>/tf</tf_topic>
-                <dimensions>2</dimensions>
-                <odom_publish_frequency>10</odom_publish_frequency>
-            </plugin>
-        </gazebo>
-    </xacro:if>
-    <!-- Lidar Config -->
-    <xacro:property name="lidar_update_rate" value="30" />
-    <xacro:property name="lidar_sample_size" value="361" />
-    <xacro:property name="lidar_min_angle" value="0" />
-    <xacro:property name="lidar_max_angle" value="360" />
-    <xacro:property name="lidar_min_range" value="0.55" />
-    <xacro:property name="lidar_max_range" value="16" />
-    <gazebo reference="lidar">
-        <sensor name='gpu_lidar' type='gpu_lidar'>
-            <topic>scan</topic>
-            <update_rate>${lidar_update_rate}</update_rate>
-            <ignition_frame_id>lidar</ignition_frame_id>
-            <lidar>
-                <scan>
-                    <horizontal>
-                        <samples>${lidar_sample_size}</samples>
-                        <resolution>1</resolution>
-                        <min_angle>${radians(lidar_min_angle)}</min_angle>
-                        <max_angle>${radians(lidar_max_angle)}</max_angle>
-                    </horizontal>
-                </scan>
-                <range>
-                    <min>${lidar_min_range}</min>
-                    <max>${lidar_max_range}</max>
-                    <resolution>0.01</resolution>
-                </range>
-                <noise>
-                    <type>gaussian</type>
-                    <mean>0.0</mean>
-                    <stddev>0.001</stddev>
-                </noise>
-            </lidar>
-            <alwaysOn>1</alwaysOn>
-            <visualize>true</visualize>
-        </sensor>
-    </gazebo>
-    <!-- Camera Config -->
-    <xacro:property name="camera_horizontal_fov" value="60" />
-    <gazebo reference="rgbd_camera_frame">
-        <sensor type="depth_camera" name="kinect_camera">
-            <update_rate>30.0</update_rate>
-            <topic>rgbd_camera</topic>
-            <ignition_frame_id>rgbd_camera_frame</ignition_frame_id>
-            <camera_info_topic>rgbd_camera_frame/camera_info</camera_info_topic>
-            <camera>
-                <horizontal_fov>${radians(camera_horizontal_fov)}</horizontal_fov>
-                <image>
-                    <width>640</width>
-                    <height>480</height>
-                    <format>R8G8B8</format>
-                </image>
-                <clip>
-                    <near>0.05</near>
-                    <far>8.0</far>
-                </clip>
-            </camera>
-        </sensor>
-    </gazebo>
-    <!-- IMU Sensor Config -->
-    <gazebo reference="imu">
-        <sensor name="imu_sensor" type="imu">
-            <always_on>1</always_on>
-            <update_rate>1</update_rate>
-            <ignition_frame_id>imu</ignition_frame_id>
-            <visualize>true</visualize>
-            <topic>imu</topic>
-        </sensor>
-    </gazebo>
-    <!-- GPS Tracker Config -->
-    <gazebo reference="gps_tracker">
-        <plugin
-            filename="ignition-gazebo-navsat-system"
-            name="ignition::gazebo::systems::NavSat">
-        </plugin>
-        <sensor name="navsat" type="navsat">
-            <always_on>1</always_on>
-            <update_rate>1</update_rate>
-            <topic>navsat</topic>
-        </sensor>
-    </gazebo>
-    <!-- Ultrasonic Sensors -->
-    <xacro:property name="us_update_rate" value="40" />
-    <xacro:property name="us_sample_size" value="11" />
-    <xacro:property name="us_min_angle" value="-7.5" />
-    <xacro:property name="us_max_angle" value="7.5" />
-    <xacro:property name="us_min_range" value="0.02" />
-    <xacro:property name="us_max_range" value="4" />
-    <xacro:macro name="us_sensor" params="frame topic">
-        <gazebo reference="${frame}">
-            <sensor name='${frame}' type='gpu_lidar'>
-                <topic>${topic}</topic>
-                <update_rate>${us_update_rate}</update_rate>
-                <ignition_frame_id>${frame}</ignition_frame_id>
-                <lidar>
-                    <scan>
-                        <horizontal>
-                            <samples>${us_sample_size}</samples>
-                            <resolution>1</resolution>
-                            <min_angle>${radians(us_min_angle)}</min_angle>
-                            <max_angle>${radians(us_max_angle)}</max_angle>
-                        </horizontal>
-                    </scan>
-                    <range>
-                        <min>${us_min_range}</min>
-                        <max>${us_max_range}</max>
-                        <resolution>0.003</resolution>
-                    </range>
-                    <noise>
-                        <type>gaussian</type>
-                        <mean>0.0</mean>
-                        <stddev>0.002</stddev>
-                    </noise>
-                </lidar>
-                <alwaysOn>1</alwaysOn>
-                <visualize>true</visualize>
-            </sensor>
-        </gazebo>
-    </xacro:macro>
-    <xacro:us_sensor frame="us_sensor_front" topic="ultrasonic/front" />
-    <xacro:us_sensor frame="us_sensor_left" topic="ultrasonic/left" />
-    <xacro:us_sensor frame="us_sensor_rear" topic="ultrasonic/rear" />
-    <xacro:us_sensor frame="us_sensor_right" topic="ultrasonic/right" />
+    <!-- DDBOT Gazebo Controllers -->
+    <xacro:include filename="$(find ddbot_gazebo)/urdf/ddbot_control.gazebo.xacro" />
+    <!-- DDBOT Gazebo Sensors -->
+    <xacro:include filename="$(find ddbot_gazebo)/urdf/ddbot_sensor.gazebo.xacro" />
 </robot>

File: ros2_ws/src/ddbot_gazebo/urdf/ddbot.xacro (robot description, xacro)
@@ -1,13 +1,10 @@
 <?xml version="1.0"?>
 <robot xmlns:xacro="http://www.ros.org/wiki/xacro" name="ddbot">
-    <xacro:arg name="wheel_odom_topic" default="odom" />
-    <xacro:arg name="odometry_source" default="world" />
-    <xacro:property name="odometry_source" value="$(arg odometry_source)" />
     <xacro:include filename="$(find ddbot_description)/urdf/ddbot.xacro" />
     <link name="base_footprint" />
     <joint name="base_footprint_joint" type="fixed">
         <origin xyz="0.0 0.0 ${base_h/2+wheel_mount_h/2+wheel_r}" rpy="0.0 0.0 0.0" />
+        <parent link="base_footprint" />
         <child link="base_link" />
-        <parent link="base_footprint" />
     </joint>
     <xacro:include filename="$(find ddbot_gazebo)/urdf/ddbot.gazebo.xacro" />
