Commit message: added imu to the simple robot description

File: ros2_ws/src/ddbot_description/urdf/ddbot.xacro (robot description, xacro)
@@ -142,5 +142,5 @@
     </link>
     <joint name="gps_tracker_joint" type="fixed">
-        <origin xyz="-${base_l/2-gps_tracker_r} 0.0 ${base_h/2+gps_tracker_l/2}" rpy="0.0 0.0 0.0" />
+        <origin xyz="-${base_l/2+gps_tracker_l/2} 0.0 0.0" rpy="0.0 -${pi/2} 0.0" />
         <parent link="base_link" />
         <child link="gps_tracker" />
@@ -186,3 +186,16 @@
         <child link="us_sensor_right" />
     </joint>
+    <!-- IMU Sensor -->
+    <xacro:property name="imu_m" value="0.05" />
+    <xacro:property name="imu_l" value="0.04" />
+    <xacro:property name="imu_w" value="0.02" />
+    <xacro:property name="imu_h" value="0.005" />
+    <link name="imu">
+        <xacro:box_link m="${imu_m}" l="${imu_l}" w="${imu_w}" h="${imu_h}" material="black" />
+    </link>
+    <joint name="imu_joint" type="fixed">
+        <origin xyz="-${base_l/4} 0.0 ${base_h/2+imu_h/2}" rpy="0.0 0.0 0.0" />
+        <parent link="base_link" />
+        <child link="imu" />
+    </joint>
 </robot>

Commit message: added sensors, robot control plugins, gui teleoperation via joystick

File: ros2_ws/src/ddbot_description/urdf/ddbot.xacro (robot description, xacro)
@@ -4,7 +4,7 @@
     <xacro:include filename="$(find ddbot_description)/urdf/link_properties.xacro" />
     <!-- Base Link -->
-    <xacro:property name="base_m" value="10" />
+    <xacro:property name="base_m" value="5.0" />
     <xacro:property name="base_l" value="0.5" />
-    <xacro:property name="base_w" value="0.35" />
+    <xacro:property name="base_w" value="0.4" />
     <xacro:property name="base_h" value="0.1" />
     <link name="base_link">
@@ -61,7 +61,7 @@
     </joint>
     <!-- Wheels -->
-    <xacro:property name="wheel_m" value="0.5" />
+    <xacro:property name="wheel_m" value="0.4" />
     <xacro:property name="wheel_r" value="0.12" />
-    <xacro:property name="wheel_l" value="0.06" />
+    <xacro:property name="wheel_l" value="0.08" />
     <link name="wheel_fl">
         <xacro:cylinder_link m="${wheel_m}" r="${wheel_r}" l="${wheel_l}" material="black" />

Commit message: added some kind of ultrasonic sensor, by utilizing lidar plugin in gazebo

File: ros2_ws/src/ddbot_description/urdf/ddbot.xacro (robot description, xacro)
@@ -149,5 +149,5 @@
     <xacro:property name="us_sensor_m" value="0.1" />
     <xacro:property name="us_sensor_r" value="0.02" />
-    <xacro:property name="us_sensor_l" value="0.06" />
+    <xacro:property name="us_sensor_l" value="0.02" />
     <link name="us_sensor_front">
         <xacro:cylinder_link m="${us_sensor_m}" r="${us_sensor_r}" l="${us_sensor_l}"
@@ -155,5 +155,5 @@
     </link>
     <joint name="us_sensor_front_joint" type="fixed">
-        <origin xyz="${base_l/2-us_sensor_l/2} 0.0 ${-base_h/2-us_sensor_r}" rpy="0.0 ${pi/2} 0.0" />
+        <origin xyz="${base_l/2-us_sensor_r} 0.0 -${base_h/2+us_sensor_l/2}" rpy="0.0 0.0 0.0" />
         <parent link="base_link" />
         <child link="us_sensor_front" />
@@ -164,5 +164,5 @@
     </link>
     <joint name="us_sensor_left_joint" type="fixed">
-        <origin xyz="0.0 ${base_w/2-us_sensor_l/2} ${-base_h/2-us_sensor_r}" rpy="${-pi/2} 0.0 0.0" />
+        <origin xyz="0.0 ${base_w/2-us_sensor_r} -${base_h/2+us_sensor_l/2}" rpy="0.0 0.0 ${pi/2}" />
         <parent link="base_link" />
         <child link="us_sensor_left" />
@@ -173,5 +173,5 @@
     </link>
     <joint name="us_sensor_rear_joint" type="fixed">
-        <origin xyz="-${base_l/2-us_sensor_l/2} 0.0 ${-base_h/2-us_sensor_r}" rpy="0.0 ${-pi/2} 0.0" />
+        <origin xyz="-${base_l/2-us_sensor_r} 0.0 -${base_h/2+us_sensor_l/2}" rpy="0.0 0.0 ${pi}" />
         <parent link="base_link" />
         <child link="us_sensor_rear" />
@@ -182,5 +182,5 @@
     </link>
     <joint name="us_sensor_right_joint" type="fixed">
-        <origin xyz="0.0 -${base_w/2-us_sensor_l/2} ${-base_h/2-us_sensor_r}" rpy="${pi/2} 0.0 0.0" />
+        <origin xyz="0.0 -${base_w/2-us_sensor_r} -${base_h/2+us_sensor_l/2}" rpy="0.0 0.0 -${pi/2}" />
         <parent link="base_link" />
         <child link="us_sensor_right" />

File: ros2_ws/src/ddbot_gazebo/urdf/ddbot.gazebo.xacro (robot description, xacro)
@@ -15,25 +15,8 @@
         <plugin filename="ignition-gazebo-diff-drive-system"
             name="ignition::gazebo::systems::DiffDrive">
+            <left_joint>wheel_fl_joint</left_joint>
+            <right_joint>wheel_fr_joint</right_joint>
             <left_joint>wheel_rl_joint</left_joint>
             <right_joint>wheel_rr_joint</right_joint>
-            <wheel_separation>${base_w+wheel_l}</wheel_separation>
-            <wheel_radius>${wheel_r}</wheel_radius>
-            <odom_publish_frequency>30</odom_publish_frequency>
-            <topic>/cmd_vel</topic>
-            <xacro:if value="${odometry_source == 'encoders'}">
-                <odom_topic>$(arg wheel_odom_topic)</odom_topic>
-                <tf_topic>/tf</tf_topic>
-            </xacro:if>
-            <max_wheel_torque>5</max_wheel_torque>
-            <max_wheel_acceleration>0.5</max_wheel_acceleration>
-            <frame_id>odom</frame_id>
-            <child_frame_id>base_footprint</child_frame_id>
-        </plugin>
-    </gazebo>
-    <gazebo>
-        <plugin filename="ignition-gazebo-diff-drive-system"
-            name="ignition::gazebo::systems::DiffDrive">
-            <left_joint>wheel_fl_joint</left_joint>
-            <right_joint>wheel_fr_joint</right_joint>
             <wheel_separation>${base_w+wheel_l}</wheel_separation>
             <wheel_radius>${wheel_r}</wheel_radius>
@@ -144,3 +127,45 @@
         </sensor>
     </gazebo>
+    <!-- Ultrasonic Sensors -->
+    <xacro:property name="us_update_rate" value="40" />
+    <xacro:property name="us_sample_size" value="11" />
+    <xacro:property name="us_min_angle" value="-7.5" />
+    <xacro:property name="us_max_angle" value="7.5" />
+    <xacro:property name="us_min_range" value="0.02" />
+    <xacro:property name="us_max_range" value="4" />
+    <xacro:macro name="us_sensor" params="frame topic">
+        <gazebo reference="${frame}">
+            <sensor name='${frame}' type='gpu_lidar'>
+                <topic>${topic}</topic>
+                <update_rate>${us_update_rate}</update_rate>
+                <ignition_frame_id>${frame}</ignition_frame_id>
+                <lidar>
+                    <scan>
+                        <horizontal>
+                            <samples>${us_sample_size}</samples>
+                            <resolution>1</resolution>
+                            <min_angle>${radians(us_min_angle)}</min_angle>
+                            <max_angle>${radians(us_max_angle)}</max_angle>
+                        </horizontal>
+                    </scan>
+                    <range>
+                        <min>${us_min_range}</min>
+                        <max>${us_max_range}</max>
+                        <resolution>0.003</resolution>
+                    </range>
+                    <noise>
+                        <type>gaussian</type>
+                        <mean>0.0</mean>
+                        <stddev>0.002</stddev>
+                    </noise>
+                </lidar>
+                <alwaysOn>1</alwaysOn>
+                <visualize>true</visualize>
+            </sensor>
+        </gazebo>
+    </xacro:macro>
+    <xacro:us_sensor frame="us_sensor_front" topic="ultrasonic/front" />
+    <xacro:us_sensor frame="us_sensor_left" topic="ultrasonic/left" />
+    <xacro:us_sensor frame="us_sensor_rear" topic="ultrasonic/rear" />
+    <xacro:us_sensor frame="us_sensor_right" topic="ultrasonic/right" />
 </robot>

Commit message: unlucky with nvsat and slam toolbox fusion

File: ros2_ws/src/ddbot_description/urdf/ddbot.xacro (robot description, xacro)
@@ -134,5 +134,5 @@
     </joint>
     <!-- GPS Tracker -->
-    <xacro:property name="gps_tracker_m" value="0.05" />
+    <xacro:property name="gps_tracker_m" value="0.1" />
     <xacro:property name="gps_tracker_r" value="0.02" />
     <xacro:property name="gps_tracker_l" value="0.02" />
@@ -147,5 +147,5 @@
     </joint>
     <!-- Ultrasonic Sensors -->
-    <xacro:property name="us_sensor_m" value="0.1" />
+    <xacro:property name="us_sensor_m" value="0.05" />
     <xacro:property name="us_sensor_r" value="0.02" />
     <xacro:property name="us_sensor_l" value="0.02" />

File: ros2_ws/src/ddbot_gazebo/urdf/ddbot_control.gazebo.xacro (robot description, xacro)
@@ -11,10 +11,10 @@
             <wheel_separation>${base_w+wheel_l}</wheel_separation>
             <wheel_radius>${wheel_r}</wheel_radius>
-            <odom_publish_frequency>30</odom_publish_frequency>
+            <odom_publish_frequency>50</odom_publish_frequency>
             <topic>/cmd_vel</topic>
             <odom_topic>/wheel/odom</odom_topic>
             <tf_topic>/wheel/tf</tf_topic>
             <max_wheel_torque>5</max_wheel_torque>
-            <max_wheel_acceleration>0.5</max_wheel_acceleration>
+            <max_wheel_acceleration>2.5</max_wheel_acceleration>
             <frame_id>odom</frame_id>
             <child_frame_id>base_footprint</child_frame_id>

File: ros2_ws/src/ddbot_gazebo/urdf/ddbot_sensor.gazebo.xacro (robot description, xacro)
@@ -41,5 +41,5 @@
     <gazebo reference="rgbd_camera_frame">
         <sensor type="depth_camera" name="kinect_camera">
-            <update_rate>30.0</update_rate>
+            <update_rate>30</update_rate>
             <topic>rgbd_camera</topic>
             <ignition_frame_id>rgbd_camera_frame</ignition_frame_id>
@@ -63,5 +63,5 @@
         <sensor name="imu_sensor" type="imu">
             <always_on>1</always_on>
-            <update_rate>25</update_rate>
+            <update_rate>50</update_rate>
             <ignition_frame_id>imu</ignition_frame_id>
             <visualize>true</visualize>
@@ -73,5 +73,5 @@
         <sensor name="navsat" type="navsat">
             <always_on>1</always_on>
-            <update_rate>10</update_rate>
+            <update_rate>5</update_rate>
             <topic>navsat</topic>
             <ignition_frame_id>gps_tracker</ignition_frame_id>
